Commit message: 完成urdf转移

File: ign_models/agibot_d1_top_description/urdf/edu.urdf (robot description, URDF)
Before this commit: robot edu_urdf, 17 links, 16 joints
Links:
- link FL_ABAD_LINK: geometry collision box size=0.1 0.07 0.07; visual mesh filename=package://agibot_d1_top_description/meshes/FL_ABAD_LINK.STL
- link FL_FOOT_LINK: geometry collision sphere radius=0.02; visual mesh filename=package://agibot_d1_top_description/meshes/FL_FOOT_LINK.STL
- link FL_HIP_LINK: geometry collision box size=0.08392 0.17199 0.25400; visual mesh filename=package://agibot_d1_top_description/meshes/FL_HIP_LINK.STL
- link FL_KNEE_LINK: geometry collision box size=0.03481 0.02000 0.11477; visual mesh filename=package://agibot_d1_top_description/meshes/FL_KNEE_LINK.STL
- link FR_ABAD_LINK: geometry collision box size=0.1 0.07 0.07; visual mesh filename=package://agibot_d1_top_description/meshes/FR_ABAD_LINK.STL
- link FR_FOOT_LINK: geometry collision sphere radius=0.02; visual mesh filename=package://agibot_d1_top_description/meshes/FR_FOOT_LINK.STL
- link FR_HIP_LINK: geometry collision box size=0.08392 0.17199 0.25400; visual mesh filename=package://agibot_d1_top_description/meshes/FR_HIP_LINK.STL
- link FR_KNEE_LINK: geometry collision box size=0.03481 0.02000 0.11477; visual mesh filename=package://agibot_d1_top_description/meshes/FR_KNEE_LINK.STL
- link RL_ABAD_LINK: geometry collision box size=0.1 0.07 0.07; visual mesh filename=package://agibot_d1_top_description/meshes/RL_ABAD_LINK.STL
- link RL_FOOT_LINK: geometry collision sphere radius=0.02; visual mesh filename=package://agibot_d1_top_description/meshes/RL_FOOT_LINK.STL
- link RL_HIP_LINK: geometry collision box size=0.08392 0.17199 0.25400; visual mesh filename=package://agibot_d1_top_description/meshes/RL_HIP_LINK.STL
- link RL_KNEE_LINK: geometry collision box size=0.03481 0.02000 0.11477; visual mesh filename=package://agibot_d1_top_description/meshes/RL_KNEE_LINK.STL
- link RR_ABAD_LINK: geometry collision box size=0.1 0.07 0.07; visual mesh filename=package://agibot_d1_top_description/meshes/RR_ABAD_LINK.STL
- link RR_FOOT_LINK: geometry collision sphere radius=0.02; visual mesh filename=package://agibot_d1_top_description/meshes/RR_FOOT_LINK.STL
- link RR_HIP_LINK: geometry collision box size=0.08392 0.17199 0.25400; visual mesh filename=package://agibot_d1_top_description/meshes/RR_HIP_LINK.STL
- link RR_KNEE_LINK: geometry collision box size=0.03481 0.02000 0.11477; visual mesh filename=package://agibot_d1_top_description/meshes/RR_KNEE_LINK.STL
- link base_link: geometry collision box size=0.4 0.1 0.05; visual mesh filename=package://agibot_d1_top_description/meshes/BASE_LINK.STL

File: ign_models/agibot_d1_top_description/urdf/top.urdf (robot description, URDF)
Before this commit: robot top.SLDASM, 5 links, 4 joints
Links:
- added link laser_device_frame
- link base_link_top: geometry visual mesh filename=package://agibot_d1_top_description/meshes/base_link_top.STL
- link camera: geometry visual mesh filename=package://agibot_d1_top_description/meshes/camera.STL
- link laser: geometry visual mesh filename=package://agibot_d1_top_description/meshes/laser.STL
Joints:
- added joint laser_device_frame_joint: type fixed, parent laser, child laser_device_frame, origin xyz=0 0 0 rpy=0 0 0
- joint laser_up_joint: origin xyz=0 0 0 rpy=0 0 0 -> xyz=0.0 0 0.1 rpy=0 0 0; parent laser -> base_link

File: src/sim_dog/agibot_d1_top_description/urdf/top.urdf (robot description, URDF)
Before this commit: robot top.SLDASM, 5 links, 4 joints
Links:
- added link laser_device_frame
- link base_link_top: geometry visual mesh filename=package://agibot_d1_top_description/meshes/base_link_top.STL
- link camera: geometry visual mesh filename=package://agibot_d1_top_description/meshes/camera.STL
- link laser: geometry visual mesh filename=package://agibot_d1_top_description/meshes/laser.STL
Joints:
- added joint laser_device_frame_joint: type fixed, parent laser, child laser_device_frame, origin xyz=0 0 0 rpy=0 0 0
- joint laser_up_joint: origin xyz=0 0 0 rpy=0 0 0 -> xyz=0.0 0 0.15 rpy=0 0 0; parent laser -> base_link
