Commit message: 优化工作空间

File: src/sim_dog/agibot_d1_top_description/urdf/edu.urdf (robot description, URDF)
Before this commit: robot edu_urdf, 17 links, 16 joints
Links:
- removed link FL_ABAD_LINK
- removed link FL_FOOT_LINK
- removed link FL_HIP_LINK
- removed link FL_KNEE_LINK
- removed link FR_ABAD_LINK
- removed link FR_FOOT_LINK
- removed link FR_HIP_LINK
- removed link FR_KNEE_LINK
- removed link RL_ABAD_LINK
- removed link RL_FOOT_LINK
- removed link RL_HIP_LINK
- removed link RL_KNEE_LINK
- removed link RR_ABAD_LINK
- removed link RR_FOOT_LINK
- removed link RR_HIP_LINK
- removed link RR_KNEE_LINK
- removed link base_link
Joints:
- removed joint FL_ABAD_JOINT
- removed joint FL_FOOT_JOINT
- removed joint FL_HIP_JOINT
- removed joint FL_KNEE_JOINT
- removed joint FR_ABAD_JOINT
- removed joint FR_FOOT_JOINT
- removed joint FR_HIP_JOINT
- removed joint FR_KNEE_JOINT
- removed joint RL_ABAD_JOINT
- removed joint RL_FOOT_JOINT
- removed joint RL_HIP_JOINT
- removed joint RL_KNEE_JOINT
- removed joint RR_ABAD_JOINT
- removed joint RR_FOOT_JOINT
- removed joint RR_HIP_JOINT
- removed joint RR_KNEE_JOINT

File: src/sim_dog/edu_description/urdf/edu.urdf (robot description, URDF)
Before this commit: robot edu_urdf, 20 links, 19 joints
Links:
- removed link front_camera
- removed link laser
- removed link laser_up
Joints:
- removed joint front_camera_joint
- removed joint laser_joint
- removed joint laser_up_joint
